File: ATTINY Reed switch.brd (EAGLE design)
At the start: 41 x 75.5 mm, 40 parts

Commit message: Add files via upload
Parts:
- removed E$19, E$20, E$21, E$22: (no value), eagle-ltspice:R0805
Routing:
- net GND6: track 2.50 -> 0.00 mm
- net GND3: track 2.50 -> 0.00 mm
- net GND2: track 2.50 -> 0.00 mm
- net GND: track 43.1 -> 40.6 mm
Changed lines of the file:
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@@
 <wire x1="41.5" y1="1" x2="40.5" y2="0" width="0.1" layer="20" curve="-90"/>
 <wire x1="40.5" y1="75.5" x2="41.5" y2="74.5" width="0.1" layer="20" curve="-90"/>
-<text x="29.17150625" y="12.381203125" size="0.6096" layer="26" font="vector" rot="SMR180">10K</text>
-<text x="12.67150625" y="24.881203125" size="0.6096" layer="26" font="vector" rot="SMR0">10K</text>
-<text x="12.67150625" y="62.881203125" size="0.6096" layer="26" font="vector" rot="SMR0">10K</text>
-<text x="29.17150625" y="50.381203125" size="0.6096" layer="26" font="vector" rot="SMR180">10K</text>
 </plain>
 <attributes>
@@
 <attribute name="VALUE" x="40.67890625" y="30.842153125" size="0.0254" layer="27" rot="R180"/>
 </element>
-<element name="E$19" library="eagle-ltspice" package="R0805" value="" x="11.854221875" y="61.354765625" smashed="yes" rot="MR0">
-<attribute name="VALUE" x="12.489221875" y="58.814765625" size="1.27" layer="28" rot="MR0"/>
-</element>
-<element name="E$20" library="eagle-ltspice" package="R0805" value="" x="11.854221875" y="23.354765625" smashed="yes" rot="MR0">
-<attribute name="VALUE" x="12.489221875" y="20.814765625" size="1.27" layer="28" rot="MR0"/>
-</element>
-<element name="E$21" library="eagle-ltspice" package="R0805" value="" x="30.145778125" y="52.145234375" smashed="yes" rot="MR180">
-<attribute name="VALUE" x="29.510778125" y="54.685234375" size="1.27" layer="28" rot="MR180"/>
-</element>
-<element name="E$22" library="eagle-ltspice" package="R0805" value="" x="30.145778125" y="13.645234375" smashed="yes" rot="MR180">
-<attribute name="VALUE" x="29.510778125" y="16.185234375" size="1.27" layer="28" rot="MR180"/>
-</element>
 </elements>
 <signals>
@@
 <wire x1="12.322734375" y1="10.386090625" x2="12.30851875" y2="10.386090625" width="0.4064" layer="16"/>
 <wire x1="12.30851875" y1="10.386090625" x2="12.30851875" y2="8.524659375" width="0.4064" layer="16"/>
-<wire x1="13" y1="61.5" x2="15.5" y2="61.5" width="0.6096" layer="16"/>
 <wire x1="9.005478125" y1="36.090496875" x2="13" y2="61.5" width="0" layer="19" extent="1-16"/>
 <wire x1="10.98869375" y1="31.071734375" x2="9.051009375" y2="31.854153125" width="0" layer="19" extent="1-1"/>
@@
 </signal>
 <signal name="GND2">
-<wire x1="13" y1="23.5" x2="15.5" y2="23.5" width="0.6096" layer="16"/>
 <wire x1="9.005478125" y1="-1.909503125" x2="13" y2="23.5" width="0" layer="19" extent="1-16"/>
 </signal>
-<signal name="GND3">
-<wire x1="29" y1="52" x2="26.5" y2="52" width="0.6096" layer="16"/>
-</signal>
-<signal name="GND6">
-<wire x1="29" y1="13.5" x2="26.5" y2="13.5" width="0.6096" layer="16"/>
-</signal>
 </signals>
